File: brain/Brain.kicad_pcb (KiCad board)
At the start: 2 copper layers, 201.5 x 128.5 mm, 103 parts, among them J1 Drive Train H-Bridge, J10 Encoder A Bypass, J2 Arm & Shooter Lazy-Suzan H-Br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, J3 Battery Connection 9V, J4 PB 5V, J5 Encoder B Bypass, J6 ESP Headers left, J7 ESP Headers right, J8 Hall Effect Sensors, J9 External Blinky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

Commit message: ready for publication, remove CI
Other:
- rule pad_to_mask_clearance: 0 -> 0.038
- board text added: "0.0000 mm / 0.0000 mm"
- board text added: "0.3000 mm"
- board text added: "1.6000 mm"
- board text added: "2"
- board text added: "201.5000 mm x 128.5000 mm"
- board text added: "BOARD CHARACTERISTICS"
- board text added: "Board Thickness:"
- board text added: "Board overall dimensions:"
- board text added: "Castellated pads:"
- board text added: "Copper Finish:"
- board text added: "Copper Layer Count:"
- board text added: "Edge card connectors:"
- board text added: "Impedance Control:"
- board text added: "Min hole diameter:"
- board text added: "Min track/spacing:"
- board text added: "No"
- board text added: "None"
- board text added: "Plated Board Edge:"
