File: brain/Brain.kicad_sch (KiCad schematic)
At the start: 57 parts, among them J1 Drive Train H-Bridge, J10 Encoder A Bypass, J2 Arm & Shooter Lazy-Suzan H-Br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, J3 Battery Connection 9V, J4 PB 5V, J5 Encoder B Bypass, J6 ESP Headers left, J7 ESP Headers right, J8 Hall Effect Sensors, J9 External Blinky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

Commit message: ready for publication, remove CI
Other:
- note added: "Random Stuff"
- note removed: "Random Shit"
Changed lines of the file:
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@@
 		(rev "Rev 1")
 		(company "The Rolling Ohms")
+		(comment 1 "Team 6 - ENPH 253 2025")
 	)
 	(text "POTS"
@@
 		)
 	)
-	(text "Random Shit"
+	(text "Random Stuff"
 		(exclude_from_sim no)
 		(at 264.922 137.922 0)
