File: brain/master_debounce.kicad_sch (KiCad schematic)
At the start: 9 parts, among them U9 LM311

Commit message: ready for publication, remove CI
Other:
- company: (none) -> The Rolling Ohms
- title: (none) -> Brain Board
Changed lines of the file:
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@@
 	(generator "eeschema")
 	(generator_version "9.0")
-	(paper "A4")
+	(paper "A3")
+	(title_block
+		(title "Brain Board")
+		(date "2025-07-08")
+		(rev "Rev 1")
+		(company "The Rolling Ohms")
+		(comment 1 "Team 6 - ENPH 253 2025")
+	)
 	(junction
 		(at 138.43 73.66)
