File: h-bridge/h_brige.kicad_sch (KiCad schematic)
At the start: 5 parts, among them U16 IRFZ44EPBF, U17 IRFZ44EPBF, U18 IRFZ44EPBF, U19 IRFZ44EPBF

Commit message: ready for publication, remove CI
Other:
- company: (none) -> The Rolling Ohms
- title: (none) -> H Bridge
Changed lines of the file:
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@@
 	(generator_version "9.0")
 	(paper "A4")
+	(title_block
+		(title "H Bridge")
+		(date "2025-07-15")
+		(rev "Rev 2")
+		(company "The Rolling Ohms")
+		(comment 1 "Team 6 ENPH 253 2025")
+	)
 	(junction
 		(at 119.38 121.92)
