File: power-distribution/Power_Board.kicad_sch (KiCad schematic)
At the start: 22 parts, among them J1 Conn_01x02, J11 Conn_01x02, J12 Conn_01x02, J15 Conn_01x02, J17 Conn_01x02, J18 Conn_01x02, J19 Conn_01x02, J2 Conn_01x02, J20 Conn_01x02, J3 Conn_01x02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

Commit message: ready for publication, remove CI
Other:
- company: (none) -> The Rolling Ohms
- title: (none) -> Power Distribution Board
- moved on the sheet: C1, C2, C3, C4, C5, C6, H1, H2, J1, J11, J12, J15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
